File: Sweep half-swept/half-swept.kicad_pcb (KiCad board)
At the start: 2 copper layers, 109.7 x 87.3 mm, 25 parts, among them J1 AudioJack4dpb, SW1 SW_Push, SW10 SW_Push, SW11 SW_Push, SW12 SW_Push, SW13 SW_Push, SW14 SW_Push, SW15 SW_Push, SW16 SW_Push, SW17 SW_Push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

Commit message: PCB update
missing pull-up resistor added to one wire serial
Parts:
- added R1: 5k6, Blackpill:0603 resistor, F.Cu at (119.4, 78.7)
Connections:
- U1 pad 38: unconnected-(U1-B14-Pad38) -> ps2_data
- U1 pad 39: unconnected-(U1-B13-Pad39) -> ps2_clk
Routing:
- net vcc: track 64.2 -> 70.0 mm
- net data: track 48.7 -> 53.6 mm
