File: Sweep half-swept/half-swept.kicad_sch (KiCad schematic)
At the start: 21 parts, among them J1 AudioJack4dpb, SW1 SW_Push, SW10 SW_Push, SW11 SW_Push, SW12 SW_Push, SW13 SW_Push, SW14 SW_Push, SW15 SW_Push, SW16 SW_Push, SW17 SW_Push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

Commit message: PCB update
missing pull-up resistor added to one wire serial
Parts:
- added R1: 5k6, Blackpill:0603 resistor, symbol Device:R
Connections:
- net data: now also R1.1
- net vcc: now also R1.2
Other:
- note added: "Pullup resistor for one wire UART"
